File: Schematics/actuator-health/actuator-health.kicad_sch (KiCad schematic)
At the start: 25 parts, among them J1 AFG connection, J2 PSU 5V connection, J3 Scope CH1, J4 Scope CH2, U1 MCP6022, U2 Pololu_4048_ACS724_05AU

Commit message: KiCad schematic work before sync
Parts:
- added C12: 4.7nF, symbol Device:C
- R1: Measured (none) -> 98.8kΩ
- R2, R3, R6: Measured (none) -> 98.9kΩ
- R4: Measured (none) -> 98.6kΩ
- R5: Measured (none) -> 216Ω
- R7: Measured (none) -> 99kΩ
- R8: value 68.8Ω -> 68Ω; Measured (none) -> 67Ω
Connections:
- net GND: now also C12.2
- net at U2.6 (FILTER): now also C12.1
- no-connect marks 1 -> 0
Other:
- moved on the sheet: J4
