File: Schematics/actuator-health/actuator-health.kicad_sch (KiCad schematic)
At the start: 23 parts, among them J1 AFE TEST / AFG, J2 5V_MEAS supply, J3 UNO R4 A0, U1 MCP6022, U2 Pololu_4048_ACS724_05AU

Commit message: Schematics fixes update
Parts:
- C3: value 1.2 nF -> 1.0 nF
- R1, R2: value 9.76k -> 10k
- R3, R4: value 4.07k -> 4.7k
Other:
- moved on the sheet: TP2
Changed lines of the file:
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@@
 	)
 	(junction
-		(at 191.77 40.64)
+		(at 254 153.67)
 		(diameter 0)
 		(color 0 0 0 0)
 	)
 	(junction
-		(at 254 153.67)
+		(at 191.77 40.64)
 		(diameter 0)
 		(color 0 0 0 0)
@@
 	(wire
 		(pts
-			(xy 195.58 31.75) (xy 195.58 40.64)
+			(xy 191.77 31.75) (xy 191.77 40.64)
 		)
 		(stroke
@@
 	(wire
 		(pts
-			(xy 191.77 40.64) (xy 195.58 40.64)
-		)
-		(stroke
-			(width 0)
-			(type default)
-		)
-	)
-	(wire
-		(pts
 			(xy 137.16 148.59) (xy 147.32 148.59)
 		)
@@
 			)
 		)
-		(property "Value" "4.07k"
+		(property "Value" "4.7k"
 			(at 60.96 134.62 90)
 			(show_name no)
@@
 			)
 		)
-		(property "Value" "4.07k"
+		(property "Value" "4.7k"
 			(at 36.83 134.62 90)
 			(show_name no)
@@
 	(symbol
 		(lib_id "Connector:TestPoint")
-		(at 195.58 31.75 0)
+		(at 191.77 31.75 0)
 		(unit 1)
 		(body_style 1)
@@
 		(fields_autoplaced yes)
 		(property "Reference" "TP2"
-			(at 198.12 27.1779 0)
+			(at 194.31 27.1779 0)
 			(show_name no)
 			(do_not_autoplace no)
@@
 		)
 		(property "Value" "TP_GND"
-			(at 198.12 29.7179 0)
+			(at 194.31 29.7179 0)
 			(show_name no)
 			(do_not_autoplace no)
@@
 		)
 		(property "Footprint" ""
-			(at 200.66 31.75 0)
+			(at 196.85 31.75 0)
 			(hide yes)
 			(show_name no)
@@
 		)
 		(property "Datasheet" ""
-			(at 200.66 31.75 0)
+			(at 196.85 31.75 0)
 			(hide yes)
 			(show_name no)
@@
 		)
 		(property "Description" "test point"
-			(at 195.58 31.75 0)
+			(at 191.77 31.75 0)
 			(hide yes)
 			(show_name no)
@@
 		(dnp no)
 		(property "Reference" "R1"
-			(at 214.63 57.15 90)
+			(at 206.756 68.834 90)
 			(show_name no)
 			(do_not_autoplace no)
@@
 			)
 		)
-		(property "Value" "9.76k"
+		(property "Value" "10k"
 			(at 207.01 71.12 90)
 			(show_name no)
@@
 			)
 		)
-		(property "Value" "9.76k"
+		(property "Value" "10k"
 			(at 231.14 63.5 90)
 			(show_name no)
@@
 			)
 		)
-		(property "Value" "1.2 nF"
+		(property "Value" "1.0 nF"
 			(at 227.33 41.9099 0)
 			(show_name no)
